File: KiCad/DBDelay _top.kicad_pcb (KiCad board)
At the start: 2 copper layers, 67.9 x 100 mm, 2 parts

Commit message: Update DBDelay _top.kicad_pcb
Parts:
- removed G***: LOGO, myFoot:dbDelay
Other:
- board text added: "DB Delay"
